File: kicad/board/board.kicad_pcb (KiCad board)
At the start: 2 copper layers, 138 x 79.2 mm, 45 parts

Commit message: undid a bunch of things in preperation for the club
Connections:
- D1 pad 1: P2 -> (no net)
- D1 pad 2: outer_bottom -> (no net)
- D1 pad 50: P2 -> (no net)
- D10 pad 1: P2 -> (no net)
- D10 pad 2: middle_bottom -> (no net)
- D10 pad 50: P2 -> (no net)
- D11 pad 1: P1 -> (no net)
- D11 pad 2: middle_home -> (no net)
- D11 pad 50: P1 -> (no net)
- D12 pad 1: P0 -> (no net)
- D12 pad 2: middle_top -> (no net)
- D12 pad 50: P0 -> (no net)
- D13 pad 1: P2 -> (no net)
- D13 pad 2: index_bottom -> (no net)
- D13 pad 50: P2 -> (no net)
- D14 pad 1: P1 -> (no net)
- D14 pad 2: index_home -> (no net)
- D14 pad 50: P1 -> (no net)
- D15 pad 1: P0 -> (no net)
- D15 pad 2: index_top -> (no net)
- D15 pad 50: P0 -> (no net)
- D16 pad 1: P2 -> (no net)
- D16 pad 2: inner_bottom -> (no net)
- D16 pad 50: P2 -> (no net)
- D17 pad 1: P1 -> (no net)
- D17 pad 2: inner_home -> (no net)
- D17 pad 50: P1 -> (no net)
- D18 pad 1: P0 -> (no net)
- D18 pad 2: inner_top -> (no net)
- D18 pad 50: P0 -> (no net)
- D19 pad 1: P7 -> (no net)
- D19 pad 2: near_thumb -> (no net)
- D19 pad 50: P7 -> (no net)
- D2 pad 1: P1 -> (no net)
- D2 pad 2: outer_home -> (no net)
- D2 pad 50: P1 -> (no net)
- D20 pad 1: P7 -> (no net)
- D20 pad 2: home_thumb -> (no net)
- D20 pad 50: P7 -> (no net)
- D21 pad 1: P7 -> (no net)
- D21 pad 2: far_thumb -> (no net)
- D21 pad 50: P7 -> (no net)
- D3 pad 1: P0 -> (no net)
- D3 pad 2: outer_top -> (no net)
- D3 pad 50: P0 -> (no net)
- D4 pad 1: P2 -> (no net)
- D4 pad 2: pinky_bottom -> (no net)
- D4 pad 50: P2 -> (no net)
- D5 pad 1: P1 -> (no net)
- D5 pad 2: pinky_home -> (no net)
- D5 pad 50: P1 -> (no net)
- D6 pad 1: P0 -> (no net)
- D6 pad 2: pinky_top -> (no net)
- D6 pad 50: P0 -> (no net)
- D7 pad 1: P2 -> (no net)
- D7 pad 2: ring_bottom -> (no net)
- D7 pad 50: P2 -> (no net)
- D8 pad 1: P1 -> (no net)
- D8 pad 2: ring_home -> (no net)
- D8 pad 50: P1 -> (no net)
- D9 pad 1: P0 -> (no net)
- D9 pad 2: ring_top -> (no net)
- D9 pad 50: P0 -> (no net)
- JST1 pad 1: BPOS -> (no net)
- JST1 pad 2: BNEG -> (no net)
- JST2 pad 1: BPOS -> (no net)
- JST2 pad 2: BNEG -> (no net)
- S1 pad 1: P3 -> (no net)
- S1 pad 2: outer_bottom -> (no net)
- S10 pad 1: P10 -> (no net)
- S10 pad 2: middle_bottom -> (no net)
- S11 pad 1: P10 -> (no net)
- S11 pad 2: middle_home -> (no net)
- S12 pad 1: P10 -> (no net)
- S12 pad 2: middle_top -> (no net)
- S13 pad 1: P9 -> (no net)
- S13 pad 2: index_bottom -> (no net)
- S14 pad 1: P9 -> (no net)
- S14 pad 2: index_home -> (no net)
- S15 pad 1: P9 -> (no net)
- S15 pad 2: index_top -> (no net)
- S16 pad 1: P8 -> (no net)
- S16 pad 2: inner_bottom -> (no net)
- S17 pad 1: P8 -> (no net)
- S17 pad 2: inner_home -> (no net)
- S18 pad 1: P8 -> (no net)
- S18 pad 2: inner_top -> (no net)
- S19 pad 1: P10 -> (no net)
- S19 pad 2: near_thumb -> (no net)
- S2 pad 1: P3 -> (no net)
- S2 pad 2: outer_home -> (no net)
- S20 pad 1: P9 -> (no net)
- S20 pad 2: home_thumb -> (no net)
- S21 pad 1: P8 -> (no net)
- S21 pad 2: far_thumb -> (no net)
- S3 pad 1: P3 -> (no net)
- S3 pad 2: outer_top -> (no net)
- S4 pad 1: P4 -> (no net)
- S4 pad 2: pinky_bottom -> (no net)
- S5 pad 1: P4 -> (no net)
- S5 pad 2: pinky_home -> (no net)
- S6 pad 1: P4 -> (no net)
- S6 pad 2: pinky_top -> (no net)
- S7 pad 1: P5 -> (no net)
- S7 pad 2: ring_bottom -> (no net)
- S8 pad 1: P5 -> (no net)
- S8 pad 2: ring_home -> (no net)
- S9 pad 1: P5 -> (no net)
- S9 pad 2: ring_top -> (no net)
Routing:
- net P10: track 173.9 -> 0.00 mm
- net P3: track 167.5 -> 0.00 mm
- net P9: track 153.4 -> 0.00 mm
- net P4: track 146.1 -> 0.00 mm
- net P8: track 143.0 -> 0.00 mm
- net P2: track 149.7 -> 10.3 mm
- net P5: track 127.0 -> 0.00 mm
- net P1: track 137.0 -> 10.3 mm
- net P0: track 127.6 -> 10.3 mm
- net P7: track 82.9 -> 0.00 mm
- net outer_top: track 26.8 -> 0.00 mm
- net outer_home: track 26.8 -> 0.00 mm
- net outer_bottom: track 26.8 -> 0.00 mm
- net near_thumb: track 26.8 -> 0.00 mm
- net inner_top: track 26.8 -> 0.00 mm
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